File: tutorials/christmas_bauble/christmas_bauble.sch (KiCad schematic (older format))
At the start: 18 parts

Commit message: Added pull down resistors. Now video 1 is complete
Parts:
- added R? (x2): 10K, symbol Device:R_US
Connections:
- net GND: now also R?.2, R?.2
- net XOR_IN_A: now also R?.1
- net XOR_IN_B: now also R?.1
Changed lines of the file:
@@
 	1400 4300 2800 4300
 Wire Wire Line
-	700  2100 1400 2100
+	700  2100 1100 2100
 Connection ~ 1400 2100
 Wire Wire Line
 	1400 2100 1650 2100
 Wire Wire Line
-	750  3600 1250 3600
+	750  3600 1100 3600
 Wire Wire Line
 	1250 3600 1250 4650
@@
 Wire Wire Line
 	5550 3300 6150 3300
+$Comp
+L Device:R_US R?
+U 1 1 606DC0E5
+P 1100 2300
+F 0 "R?" V 895 2300 50  0000 C CNN
+F 1 "10K" V 986 2300 50  0000 C CNN
+F 2 "" V 1140 2290 50  0001 C CNN
+F 3 "~" H 1100 2300 50  0001 C CNN
+	1    1100 2300
+	1    0    0    -1
+$EndComp
+$Comp
+L Device:R_US R?
+U 1 1 606DD704
+P 1100 3800
+F 0 "R?" V 895 3800 50  0000 C CNN
+F 1 "10K" V 986 3800 50  0000 C CNN
+F 2 "" V 1140 3790 50  0001 C CNN
+F 3 "~" H 1100 3800 50  0001 C CNN
+	1    1100 3800
+	1    0    0    -1
+$EndComp
+Wire Wire Line
+	1100 2100 1100 2150
+Connection ~ 1100 2100
+Wire Wire Line
+	1100 2100 1400 2100
+$Comp
+L power:GND #PWR?
+U 1 1 606E1B79
+P 1100 2550
+F 0 "#PWR?" H 1100 2300 50  0001 C CNN
+F 1 "GND" H 1105 2377 50  0000 C CNN
+F 2 "" H 1100 2550 50  0001 C CNN
+F 3 "" H 1100 2550 50  0001 C CNN
+	1    1100 2550
+	1    0    0    -1
+$EndComp
+$Comp
+L power:GND #PWR?
+U 1 1 606E3093
+P 1100 4000
+F 0 "#PWR?" H 1100 3750 50  0001 C CNN
+F 1 "GND" H 1105 3827 50  0000 C CNN
+F 2 "" H 1100 4000 50  0001 C CNN
+F 3 "" H 1100 4000 50  0001 C CNN
+	1    1100 4000
+	1    0    0    -1
+$EndComp
+Wire Wire Line
+	1100 2450 1100 2550
+Wire Wire Line
+	1100 3600 1100 3650
+Connection ~ 1100 3600
+Wire Wire Line
+	1100 3600 1250 3600
+Wire Wire Line
+	1100 3950 1100 4000
 $EndSCHEMATC
