File: hw/designs/stm32_breakout/_autosave-stm32_breakout.sch (KiCad schematic (older format))
At the start: 20 parts, among them J1 USB_B_Micro, J2 Conn_01x10_Male, J3 Conn_01x10_Male, J4 Conn_01x03_Male, U1 AP7361C-33E, U2 STM32L031F6Px, U3 KC2016Z, Y1 ABS25-32.768KHZ-6-T

Commit message: Removed RTC circuit. Changed pinout on headers. Updated jumpers to resistors instead. Started routing
Parts:
- removed C1, C2: 4.3pF, Capacitor_SMD:C_0805_2012Metric, symbol pspice:CAP
- removed J4: Conn_01x03_Male, Connector_PinSocket_2.54mm:PinSocket_1x03_P2.54mm_Vertical, symbol Connector:Conn_01x03_Male
- removed JP1, JP2: Jumper, Connector_PinSocket_2.54mm:PinSocket_1x02_P2.54mm_Vertical, symbol Device:Jumper
- removed Y1: ABS25-32.768KHZ-6-T, Custom:XTAL_ABS25-32.768KHZ-6-1-T, symbol Device:Crystal_GND23
- added R2: 0, Resistor_SMD:R_0805_2012Metric, symbol Device:R_US
- added R3: UNPOP, Resistor_SMD:R_0805_2012Metric, symbol Device:R_US
- renumbered C3 to C1, C4 to C2, C5 to C3, C6 to C4, C7 to C5, C8 to C6
Connections:
- net +3V3: now also J2.10 (Pin_10), R2.1; no longer J2.1 (Pin_1)
- net GND: now also J3.10 (Pin_10), R3.2; no longer J2.10 (Pin_10)
- net PA10: now also J2.8 (Pin_8); no longer J3.10 (Pin_10)
- net PA13: now also J2.6 (Pin_6); no longer J2.3 (Pin_3)
- net PA14: now also J2.7 (Pin_7); no longer J2.4 (Pin_4)
- net PA5: now also J3.7 (Pin_7); no longer J3.6 (Pin_6)
- net PA6: now also J3.6 (Pin_6); no longer J3.7 (Pin_7)
- net PA9: now also J2.9 (Pin_9); no longer J3.9 (Pin_9)
- net PB1: now also J3.9 (Pin_9); no longer J2.7 (Pin_7)
- net PB9-BOOT0: now also J2.5 (Pin_5); no longer J2.8 (Pin_8)
- net PC14-OSC32IN: now also J2.4 (Pin_4); no longer J2.5 (Pin_5)
- net PC15-OSC32_OUT: now also J2.3 (Pin_3); no longer J2.6 (Pin_6)
- net at U3.1 (INH): now also R2.2, R3.1
- no-connect marks 8 -> 6
Other:
- note added: "Use KC2016Z: R2 = 0, R3 = UNPOP\nUse Internal Clock: R2 = UNPOP, R3 = 0"
