File: hw/designs/stm32_breakout/stm32_breakout.sch (KiCad schematic (older format))
At the start: 7 parts

Commit message: Added clocking and jumpers
Parts:
- added C? (x2): 4.3pF, symbol pspice:CAP
- added J?: Conn_01x03_Male, symbol Connector:Conn_01x03_Male
- added J? (x2): Conn_01x10_Male, symbol Connector:Conn_01x10_Male
- added JP?: Jumper, symbol Device:Jumper
- added R?: 0, symbol Device:R_US
- added U?: KC2016Z, symbol kc2016z:KC2016Z
- added Y?: ABS25-32.768KHZ-6-T, symbol Device:Crystal_GND23
Connections:
- net labels added: +3.3V
- wire segments 47 -> 100

Commit message: Updated to 32K flash and replaced resistor with jumper. Also added Nucleo reference material
Parts:
- removed R?: 0, symbol Device:R_US
- removed U?: STM32L011F3Px, Package_SO:TSSOP-20_4.4x6.5mm_P0.65mm, symbol MCU_ST_STM32L0:STM32L011F3Px
- added JP?: Jumper, symbol Device:Jumper
- added U?: STM32L031F6Px, Package_SO:TSSOP-20_4.4x6.5mm_P0.65mm, symbol MCU_ST_STM32L0:STM32L031F6Px
Other:
- moved on the sheet: JP?
Changed lines of the file:
@@
 Comment4 ""
 $EndDescr
-$Comp
-L MCU_ST_STM32L0:STM32L011F3Px U?
-U 1 1 607E1789
-P 5750 3250
-F 0 "U?" H 5700 2361 50  0000 C CNN
-F 1 "STM32L011F3Px" H 5700 2270 50  0000 C CNN
-F 2 "Package_SO:TSSOP-20_4.4x6.5mm_P0.65mm" H 5350 2550 50  0001 R CNN
-F 3 "http://www.st.com/st-web-ui/static/active/en/resource/technical/document/datasheet/DM00206508.pdf" H 5750 3250 50  0001 C CNN
-	1    5750 3250
-	1    0    0    -1
-$EndComp
 Text Label 4450 2750 0    50   ~ 0
 NRST
-Wire Wire Line
-	5250 2750 4450 2750
-Text Label 4450 3450 0    50   ~ 0
-PC14-OSC32IN
-Text Label 4450 3750 0    50   ~ 0
+Text Label 4450 3850 0    50   ~ 0
 PB1
-Wire Wire Line
-	5250 3750 4450 3750
-Text Label 4450 3850 0    50   ~ 0
+Text Label 4450 2950 0    50   ~ 0
 PB9-BOOT0
-Wire Wire Line
-	4450 3850 5250 3850
 Text Label 6700 2750 0    50   ~ 0
 PA0-CK_IN
@@
 Text Label 6700 3850 0    50   ~ 0
 PA14
-Wire Wire Line
-	6150 2850 6700 2850
-Wire Wire Line
-	6150 2950 6700 2950
-Wire Wire Line
-	6150 3050 6700 3050
-Wire Wire Line
-	6150 3150 6700 3150
-Wire Wire Line
-	6150 3250 6700 3250
-Wire Wire Line
-	6150 3350 6700 3350
-Wire Wire Line
-	6150 3450 6700 3450
-Wire Wire Line
-	6150 3550 6700 3550
-Wire Wire Line
-	6150 3650 6700 3650
-Wire Wire Line
-	6150 3750 6700 3750
-Wire Wire Line
-	6150 3850 6700 3850
 $Comp
 L power:GND #PWR?
@@
 	7150 3600 7150 2750
 Wire Wire Line
-	6150 2750 7150 2750
-Wire Wire Line
 	8850 3050 8850 3100
 $Comp
@@
 Wire Wire Line
 	8450 2800 8450 2750
-Text Label 4450 3550 0    50   ~ 0
+Text Label 4450 3650 0    50   ~ 0
 PC15-OSC32_OUT
 $Comp
@@
 $EndComp
 $Comp
-L Device:Jumper JP?
-U 1 1 60861856
-P 3300 3450
-F 0 "JP?" H 3300 3714 50  0000 C CNN
-F 1 "Jumper" H 3300 3623 50  0000 C CNN
-F 2 "" H 3300 3450 50  0001 C CNN
-F 3 "~" H 3300 3450 50  0001 C CNN
-	1    3300 3450
-	1    0    0    -1
-$EndComp
-$Comp
 L pspice:CAP C?
 U 1 1 60862421
@@
 Wire Wire Line
 	2850 3450 2550 3450
-Wire Wire Line
-	3000 3450 2850 3450
 Connection ~ 2850 3450
 Wire Wire Line
-	3150 4150 2850 4150
+	3200 4150 2850 4150
 Wire Wire Line
 	2850 4150 2850 3900
@@
 	1900 4150 2050 4150
 Wire Wire Line
-	4250 4150 4250 3550
-Wire Wire Line
-	4250 3550 5250 3550
+	4250 4150 4250 3650
 $Comp
 L power:GND #PWR?
@@
 	1900 4150 1900 4300
 Connection ~ 1900 4150
-$Comp
-L Device:R_US R?
-U 1 1 6085EB60
-P 3300 4150
-F 0 "R?" V 3095 4150 50  0000 C CNN
-F 1 "0" H 3186 4150 50  0000 C CNN
-F 2 "" V 3340 4140 50  0001 C CNN
-F 3 "~" H 3300 4150 50  0001 C CNN
-	1    3300 4150
-	0    1    1    0
-$EndComp
-Wire Wire Line
-	3600 3450 5250 3450
-Wire Wire Line
-	3450 4150 4250 4150
 $Comp
 L Connector:Conn_01x10_Male J?
@@
 	3750 5150 3150 5150
 Wire Wire Line
-	3150 5850 3500 5850
-Wire Wire Line
 	3500 5950 3150 5950
 $Comp
@@
 	3500 5950 3500 6150
 Wire Wire Line
-	3500 5850 3500 5950
-Connection ~ 3500 5950
-Wire Wire Line
 	6400 5000 6950 5000
+$Comp
+L Device:Jumper JP?
+U 1 1 60875E00
+P 3500 4150
+F 0 "JP?" H 3500 4414 50  0000 C CNN
+F 1 "Jumper" H 3500 4323 50  0000 C CNN
+F 2 "" H 3500 4150 50  0001 C CNN
+F 3 "~" H 3500 4150 50  0001 C CNN
+	1    3500 4150
+	1    0    0    -1
+$EndComp
+$Comp
+L MCU_ST_STM32L0:STM32L031F6Px U?
+U 1 1 6087A076
+P 5650 3250
+F 0 "U?" H 5650 2361 50  0000 C CNN
+F 1 "STM32L031F6Px" H 5650 2270 50  0000 C CNN
+F 2 "Package_SO:TSSOP-20_4.4x6.5mm_P0.65mm" H 5250 2550 50  0001 R CNN
+F 3 "http://www.st.com/st-web-ui/static/active/en/resource/technical/document/datasheet/DM00140359.pdf" H 5650 3250 50  0001 C CNN
+	1    5650 3250
+	1    0    0    -1
+$EndComp
+Wire Wire Line
+	4250 4150 3800 4150
+Wire Wire Line
+	6150 2750 7150 2750
+Wire Wire Line
+	6150 3850 6700 3850
+Wire Wire Line
+	6150 3750 6700 3750
+Wire Wire Line
+	6150 3650 6700 3650
+Wire Wire Line
+	6150 3550 6700 3550
+Wire Wire Line
+	6150 3450 6700 3450
+Wire Wire Line
+	6150 3350 6700 3350
+Wire Wire Line
+	6150 3250 6700 3250
+Wire Wire Line
+	6150 3150 6700 3150
+Wire Wire Line
+	6150 3050 6700 3050
+Wire Wire Line
+	6150 2950 6700 2950
+Wire Wire Line
+	6150 2850 6700 2850
+Wire Wire Line
+	3200 3450 2850 3450
+$Comp
+L Device:Jumper JP?
+U 1 1 60861856
+P 3500 3450
+F 0 "JP?" H 3500 3714 50  0000 C CNN
+F 1 "Jumper" H 3500 3623 50  0000 C CNN
+F 2 "" H 3500 3450 50  0001 C CNN
+F 3 "~" H 3500 3450 50  0001 C CNN
+	1    3500 3450
+	1    0    0    -1
+$EndComp
+Text Label 4450 3550 0    50   ~ 0
+PC14-OSC32IN
+Wire Wire Line
+	4450 2950 5150 2950
+Wire Wire Line
+	4250 3650 5150 3650
+Wire Wire Line
+	3800 3450 4250 3450
+Wire Wire Line
+	5150 3550 4250 3550
+Wire Wire Line
+	4250 3550 4250 3450
+Wire Wire Line
+	4450 3850 5150 3850
+Wire Wire Line
+	5150 2750 4450 2750
 $EndSCHEMATC

Commit message: Added bypass caps to the voltage regulator.
Parts:
- added C?: 4.7u, symbol pspice:C
- added C?: 4.7u, symbol pspice:CAP
- J?: symbol Connector:USB_B_Micro -> stm32_breakout-rescue:USB_B_Micro-Connector
- U?: symbol kc2016z:KC2016Z -> stm32_breakout-rescue:KC2016Z-kc2016z
Connections:
- wire segments 100 -> 109
Changed lines of the file:
@@
 Wire Wire Line
 	5300 2200 5300 2400
-Connection ~ 5300 2400
-Wire Wire Line
-	5300 2400 4850 2400
 Wire Wire Line
 	5300 1700 5300 1500
@@
 $EndComp
 Wire Wire Line
-	3300 2400 3750 2400
-Wire Wire Line
 	5650 2400 5650 2550
-Connection ~ 4850 2400
 $Comp
 L power:GND #PWR?
@@
 	3000 2700 3000 2900
 $Comp
-L Connector:USB_B_Micro J?
+L stm32_breakout-rescue:USB_B_Micro-Connector J?
 U 1 1 60814F1F
 P 1850 2600
@@
 Connection ~ 1800 3100
 Wire Wire Line
-	2700 2400 2150 2400
+	2700 2400 2500 2400
 Wire Wire Line
 	7150 3600 7150 2750
@@
 	8850 2450 8850 2400
 $Comp
-L kc2016z:KC2016Z U?
+L stm32_breakout-rescue:KC2016Z-kc2016z U?
 U 1 1 6081180B
 P 8850 2750
@@
 L power:+3.3V #PWR?
 U 1 1 60904649
-P 3750 2150
-F 0 "#PWR?" H 3750 2000 50  0001 C CNN
-F 1 "+3.3V" H 3765 2323 50  0000 C CNN
-F 2 "" H 3750 2150 50  0001 C CNN
-F 3 "" H 3750 2150 50  0001 C CNN
-	1    3750 2150
-	1    0    0    -1
-$EndComp
-Wire Wire Line
-	3750 2150 3750 2400
-Connection ~ 3750 2400
-Wire Wire Line
-	3750 2400 4850 2400
+P 4000 2250
+F 0 "#PWR?" H 4000 2100 50  0001 C CNN
+F 1 "+3.3V" H 4015 2423 50  0000 C CNN
+F 2 "" H 4000 2250 50  0001 C CNN
+F 3 "" H 4000 2250 50  0001 C CNN
+	1    4000 2250
+	1    0    0    -1
+$EndComp
+Wire Wire Line
+	4000 2250 4000 2400
+Connection ~ 4000 2400
+Wire Wire Line
+	4000 2400 4850 2400
 $Comp
 L power:+3.3V #PWR?
@@
 Wire Wire Line
 	5150 2750 4450 2750
+$Comp
+L pspice:C C?
+U 1 1 60868E65
+P 2500 1900
+F 0 "C?" H 2678 1946 50  0000 L CNN
+F 1 "4.7u" H 2678 1855 50  0000 L CNN
+F 2 "" H 2500 1900 50  0001 C CNN
+F 3 "~" H 2500 1900 50  0001 C CNN
+	1    2500 1900
+	1    0    0    -1
+$EndComp
+$Comp
+L pspice:CAP C?
+U 1 1 608699C3
+P 3450 1900
+F 0 "C?" H 3628 1946 50  0000 L CNN
+F 1 "4.7u" H 3628 1855 50  0000 L CNN
+F 2 "" H 3450 1900 50  0001 C CNN
+F 3 "~" H 3450 1900 50  0001 C CNN
+	1    3450 1900
+	1    0    0    -1
+$EndComp
+Wire Wire Line
+	4850 2400 5300 2400
+Connection ~ 4850 2400
+Connection ~ 5300 2400
+Wire Wire Line
+	3300 2400 3450 2400
+Wire Wire Line
+	3450 2400 3450 2150
+Wire Wire Line
+	3450 2400 4000 2400
+Connection ~ 3450 2400
+Wire Wire Line
+	2500 2150 2500 2400
+Connection ~ 2500 2400
+Wire Wire Line
+	2500 2400 2150 2400
+Wire Wire Line
+	3450 1650 3450 1500
+Wire Wire Line
+	2500 1650 2500 1500
+$Comp
+L power:GND #PWR?
+U 1 1 608998B1
+P 4100 1700
+F 0 "#PWR?" H 4100 1450 50  0001 C CNN
+F 1 "GND" H 4105 1527 50  0000 C CNN
+F 2 "" H 4100 1700 50  0001 C CNN
+F 3 "" H 4100 1700 50  0001 C CNN
+	1    4100 1700
+	1    0    0    -1
+$EndComp
+Wire Wire Line
+	4100 1500 4100 1700
+Wire Wire Line
+	3450 1500 4100 1500
+Wire Wire Line
+	2500 1500 3450 1500
+Connection ~ 3450 1500
 $EndSCHEMATC

Commit message: Added LED, annotated schematic, and ERC is passing
Parts:
- added D1: LED, symbol Device:LED
- added R1: 200, symbol Device:R_US
- J1: renamed from J?; symbol stm32_breakout-rescue:USB_B_Micro-Connector -> stm32_breakout-rescue:USB_B_Micro-Connector-stm32_breakout-rescue
- U3: renamed from U?; symbol stm32_breakout-rescue:KC2016Z-kc2016z -> stm32_breakout-rescue:KC2016Z-kc2016z-stm32_breakout-rescue
- gave numbers to parts that had none: 16
Connections:
- net GND: now also D1.1 (K)
- net at C3.2, J1.1 (VBUS), U1.1 (VI): now also R1.2
- new net: D1.2 (A), R1.1
- no-connect marks 0 -> 8
Changed lines of the file:
@@
 PA14
 $Comp
-L power:GND #PWR?
+L power:GND #PWR0101
 U 1 1 607E9570
 P 5650 4350
-F 0 "#PWR?" H 5650 4100 50  0001 C CNN
+F 0 "#PWR0101" H 5650 4100 50  0001 C CNN
 F 1 "GND" H 5655 4177 50  0000 C CNN
 F 2 "" H 5650 4350 50  0001 C CNN
@@
 	5650 4050 5650 4350
 $Comp
-L pspice:CAP C?
+L pspice:CAP C5
 U 1 1 607E9DE9
 P 4850 1950
-F 0 "C?" H 5028 1996 50  0000 L CNN
+F 0 "C5" H 5028 1996 50  0000 L CNN
 F 1 "100nF" H 5028 1905 50  0000 L CNN
 F 2 "" H 4850 1950 50  0001 C CNN
@@
 $EndComp
 $Comp
-L pspice:CAP C?
+L pspice:CAP C7
 U 1 1 607ECA39
 P 6000 1950
-F 0 "C?" H 6178 1996 50  0000 L CNN
+F 0 "C7" H 6178 1996 50  0000 L CNN
 F 1 "100nF" H 6178 1905 50  0000 L CNN
 F 2 "" H 6000 1950 50  0001 C CNN
@@
 $EndComp
 $Comp
-L pspice:CAP C?
+L pspice:CAP C8
 U 1 1 607ECE2C
 P 6500 1950
-F 0 "C?" H 6678 1996 50  0000 L CNN
+F 0 "C8" H 6678 1996 50  0000 L CNN
 F 1 "1uF" H 6678 1905 50  0000 L CNN
 F 2 "" H 6500 1950 50  0001 C CNN
@@
 	4550 1500 4850 1500
 $Comp
-L power:GND #PWR?
+L power:GND #PWR0102
 U 1 1 607FBD40
 P 6900 1700
-F 0 "#PWR?" H 6900 1450 50  0001 C CNN
+F 0 "#PWR0102" H 6900 1450 50  0001 C CNN
 F 1 "GND" H 6905 1527 50  0000 C CNN
 F 2 "" H 6900 1700 50  0001 C CNN
@@
 	6500 1500 6000 1500
 $Comp
-L power:GND #PWR?
+L power:GND #PWR0103
 U 1 1 60806A08
 P 4550 1700
-F 0 "#PWR?" H 4550 1450 50  0001 C CNN
+F 0 "#PWR0103" H 4550 1450 50  0001 C CNN
 F 1 "GND" H 4555 1527 50  0000 C CNN
 F 2 "" H 4550 1700 50  0001 C CNN
@@
 Connection ~ 5650 2400
 $Comp
-L pspice:CAP C?
+L pspice:CAP C6
 U 1 1 607EC639
 P 5300 1950
-F 0 "C?" H 5478 1996 50  0000 L CNN
+F 0 "C6" H 5478 1996 50  0000 L CNN
 F 1 "10uF" H 5478 1905 50  0000 L CNN
 F 2 "" H 5300 1950 50  0001 C CNN
@@
 $EndComp
 $Comp
-L Regulator_Linear:AP7361C-33E U?
+L Regulator_Linear:AP7361C-33E U1
 U 1 1 608118E6
 P 3000 2400
-F 0 "U?" H 3000 2642 50  0000 C CNN
+F 0 "U1" H 3000 2642 50  0000 C CNN
 F 1 "AP7361C-33E" H 3000 2551 50  0000 C CNN
 F 2 "Package_TO_SOT_SMD:SOT-223-3_TabPin2" H 3000 2625 50  0001 C CIN
@@
 	5650 2400 5650 2550
 $Comp
-L power:GND #PWR?
+L power:GND #PWR0104
 U 1 1 60812C1A
 P 3000 2900
-F 0 "#PWR?" H 3000 2650 50  0001 C CNN
+F 0 "#PWR0104" H 3000 2650 50  0001 C CNN
 F 1 "GND" H 3005 2727 50  0000 C CNN
 F 2 "" H 3000 2900 50  0001 C CNN
@@
 	3000 2700 3000 2900
 $Comp
-L stm32_breakout-rescue:USB_B_Micro-Connector J?
+L stm32_breakout-rescue:USB_B_Micro-Connector-stm32_breakout-rescue J1
 U 1 1 60814F1F
 P 1850 2600
-F 0 "J?" H 1907 3067 50  0000 C CNN
+F 0 "J1" H 1907 3067 50  0000 C CNN
 F 1 "USB_B_Micro" H 1907 2976 50  0000 C CNN
 F 2 "" H 2000 2550 50  0001 C CNN
@@
 $EndComp
 $Comp
-L power:GND #PWR?
+L power:GND #PWR0105
 U 1 1 60817F53
 P 1800 3300
-F 0 "#PWR?" H 1800 3050 50  0001 C CNN
+F 0 "#PWR0105" H 1800 3050 50  0001 C CNN
 F 1 "GND" H 1805 3127 50  0000 C CNN
 F 2 "" H 1800 3300 50  0001 C CNN
@@
 	8850 3050 8850 3100
 $Comp
-L power:GND #PWR?
+L power:GND #PWR0106
 U 1 1 6082D318
 P 8850 3250
-F 0 "#PWR?" H 8850 3000 50  0001 C CNN
+F 0 "#PWR0106" H 8850 3000 50  0001 C CNN
 F 1 "GND" H 8855 3077 50  0000 C CNN
 F 2 "" H 8850 3250 50  0001 C CNN
@@
 	8850 2450 8850 2400
 $Comp
-L stm32_breakout-rescue:KC2016Z-kc2016z U?
+L stm32_breakout-rescue:KC2016Z-kc2016z-stm32_breakout-rescue U3
 U 1 1 6081180B
 P 8850 2750
-F 0 "U?" H 9294 2796 50  0000 L CNN
+F 0 "U3" H 9294 2796 50  0000 L CNN
 F 1 "KC2016Z" H 9294 2705 50  0000 L CNN
 F 2 "" H 9000 2900 50  0001 C CNN
@@
 	7150 3600 9700 3600
 $Comp
-L Connector:Conn_01x03_Male J?
+L Connector:Conn_01x03_Male J4
 U 1 1 6083CA4A
 P 7850 2800
-F 0 "J?" H 7958 3081 50  0000 C CNN
+F 0 "J4" H 7958 3081 50  0000 C CNN
 F 1 "Conn_01x03_Male" H 7958 2990 50  0000 C CNN
 F 2 "" H 7850 2800 50  0001 C CNN
@@
 PC15-OSC32_OUT
 $Comp
-L Device:Crystal_GND23 Y?
+L Device:Crystal_GND23 Y1
 U 1 1 60849DF1
 P 2850 3750
-F 0 "Y?" V 2804 3994 50  0000 L CNN
+F 0 "Y1" V 2804 3994 50  0000 L CNN
 F 1 "ABS25-32.768KHZ-6-T" V 2895 3994 50  0000 L CNN
 F 2 "" H 2850 3750 50  0001 C CNN
@@
 $EndComp
 $Comp
-L pspice:CAP C?
+L pspice:CAP C1
 U 1 1 60862421
 P 2300 3450
-F 0 "C?" V 1985 3450 50  0000 C CNN
+F 0 "C1" V 1985 3450 50  0000 C CNN
 F 1 "4.3pF" V 2076 3450 50  0000 C CNN
 F 2 "" H 2300 3450 50  0001 C CNN
@@
 $EndComp
 $Comp
-L pspice:CAP C?
+L pspice:CAP C2
 U 1 1 608657C5
 P 2300 4150
-F 0 "C?" V 1985 4150 50  0000 C CNN
+F 0 "C2" V 1985 4150 50  0000 C CNN
 F 1 "4.3pF" V 2076 4150 50  0000 C CNN
 F 2 "" H 2300 4150 50  0001 C CNN
@@
 	4250 4150 4250 3650
 $Comp
-L power:GND #PWR?
+L power:GND #PWR0107
 U 1 1 60879536
 P 1900 4300
-F 0 "#PWR?" H 1900 4050 50  0001 C CNN
+F 0 "#PWR0107" H 1900 4050 50  0001 C CNN
 F 1 "GND" H 1905 4127 50  0000 C CNN
 F 2 "" H 1900 4300 50  0001 C CNN
@@
 Connection ~ 1900 4150
 $Comp
-L Connector:Conn_01x10_Male J?
+L Connector:Conn_01x10_Male J3
 U 1 1 60894859
 P 6200 5400
-F 0 "J?" H 6308 5981 50  0000 C CNN
+F 0 "J3" H 6308 5981 50  0000 C CNN
 F 1 "Conn_01x10_Male" H 6308 5890 50  0000 C CNN
 F 2 "" H 6200 5400 50  0001 C CNN
@@
 $EndComp
 $Comp
-L Connector:Conn_01x10_Male J?
+L Connector:Conn_01x10_Male J2
 U 1 1 60898F4F
 P 2950 5450
-F 0 "J?" H 3058 6031 50  0000 C CNN
+F 0 "J2" H 3058 6031 50  0000 C CNN
 F 1 "Conn_01x10_Male" H 3058 5940 50  0000 C CNN
 F 2 "" H 2950 5450 50  0001 C CNN
@@
 	3150 5750 3750 5750
 $Comp
-L power:+3.3V #PWR?
+L power:+3.3V #PWR0108
 U 1 1 60904649
 P 4000 2250
-F 0 "#PWR?" H 4000 2100 50  0001 C CNN
+F 0 "#PWR0108" H 4000 2100 50  0001 C CNN
 F 1 "+3.3V" H 4015 2423 50  0000 C CNN
 F 2 "" H 4000 2250 50  0001 C CNN
@@
 	4000 2400 4850 2400
 $Comp
-L power:+3.3V #PWR?
+L power:+3.3V #PWR0109
 U 1 1 6090C2FF
 P 3500 4850
-F 0 "#PWR?" H 3500 4700 50  0001 C CNN
+F 0 "#PWR0109" H 3500 4700 50  0001 C CNN
 F 1 "+3.3V" H 3515 5023 50  0000 C CNN
 F 2 "" H 3500 4850 50  0001 C CNN
@@
 	3500 5950 3150 5950
 $Comp
-L power:GND #PWR?
+L power:GND #PWR0110
 U 1 1 6091C1DA
 P 3500 6150
-F 0 "#PWR?" H 3500 5900 50  0001 C CNN
+F 0 "#PWR0110" H 3500 5900 50  0001 C CNN
 F 1 "GND" H 3505 5977 50  0000 C CNN
 F 2 "" H 3500 6150 50  0001 C CNN
@@
 	6400 5000 6950 5000
 $Comp
-L Device:Jumper JP?
+L Device:Jumper JP2
 U 1 1 60875E00
 P 3500 4150
-F 0 "JP?" H 3500 4414 50  0000 C CNN
+F 0 "JP2" H 3500 4414 50  0000 C CNN
 F 1 "Jumper" H 3500 4323 50  0000 C CNN
 F 2 "" H 3500 4150 50  0001 C CNN
@@
 $EndComp
 $Comp
-L MCU_ST_STM32L0:STM32L031F6Px U?
+L MCU_ST_STM32L0:STM32L031F6Px U2
 U 1 1 6087A076
 P 5650 3250
-F 0 "U?" H 5650 2361 50  0000 C CNN
+F 0 "U2" H 5650 2361 50  0000 C CNN
 F 1 "STM32L031F6Px" H 5650 2270 50  0000 C CNN
 F 2 "Package_SO:TSSOP-20_4.4x6.5mm_P0.65mm" H 5250 2550 50  0001 R CNN
@@
 	3200 3450 2850 3450
 $Comp
-L Device:Jumper JP?
+L Device:Jumper JP1
 U 1 1 60861856
 P 3500 3450
-F 0 "JP?" H 3500 3714 50  0000 C CNN
+F 0 "JP1" H 3500 3714 50  0000 C CNN
 F 1 "Jumper" H 3500 3623 50  0000 C CNN
 F 2 "" H 3500 3450 50  0001 C CNN
@@
 	5150 2750 4450 2750
 $Comp
-L pspice:C C?
+L pspice:C C3
 U 1 1 60868E65
 P 2500 1900
-F 0 "C?" H 2678 1946 50  0000 L CNN
+F 0 "C3" H 2678 1946 50  0000 L CNN
 F 1 "4.7u" H 2678 1855 50  0000 L CNN
 F 2 "" H 2500 1900 50  0001 C CNN
@@
 $EndComp
 $Comp
-L pspice:CAP C?
+L pspice:CAP C4
 U 1 1 608699C3
 P 3450 1900
-F 0 "C?" H 3628 1946 50  0000 L CNN
+F 0 "C4" H 3628 1946 50  0000 L CNN
 F 1 "4.7u" H 3628 1855 50  0000 L CNN
 F 2 "" H 3450 1900 50  0001 C CNN
@@
 Connection ~ 2500 2400
 Wire Wire Line
-	2500 2400 2150 2400
+	2500 2400 2200 2400
 Wire Wire Line
 	3450 1650 3450 1500
@@
 	2500 1650 2500 1500
 $Comp
-L power:GND #PWR?
+L power:GND #PWR0111
 U 1 1 608998B1
 P 4100 1700
-F 0 "#PWR?" H 4100 1450 50  0001 C CNN
+F 0 "#PWR0111" H 4100 1450 50  0001 C CNN
 F 1 "GND" H 4105 1527 50  0000 C CNN
 F 2 "" H 4100 1700 50  0001 C CNN
@@
 	2500 1500 3450 1500
 Connection ~ 3450 1500
+$Comp
+L Device:R_US R1
+U 1 1 60937DDE
+P 2200 1950
+F 0 "R1" H 2268 1996 50  0000 L CNN
+F 1 "200" H 2268 1905 50  0000 L CNN
+F 2 "" V 2240 1940 50  0001 C CNN
+F 3 "~" H 2200 1950 50  0001 C CNN
+	1    2200 1950
+	1    0    0    -1
+$EndComp
+$Comp
+L Device:LED D1
+U 1 1 60938A45
+P 1900 1750
+F 0 "D1" H 1893 1967 50  0000 C CNN
+F 1 "LED" H 1893 1876 50  0000 C CNN
+F 2 "" H 1900 1750 50  0001 C CNN
+F 3 "~" H 1900 1750 50  0001 C CNN
+	1    1900 1750
+	1    0    0    -1
+$EndComp
+$Comp
+L power:GND #PWR01
+U 1 1 609399D5
+P 1550 1850
+F 0 "#PWR01" H 1550 1600 50  0001 C CNN
+F 1 "GND" H 1555 1677 50  0000 C CNN
+F 2 "" H 1550 1850 50  0001 C CNN
+F 3 "" H 1550 1850 50  0001 C CNN
+	1    1550 1850
+	1    0    0    -1
+$EndComp
+Wire Wire Line
+	2200 2100 2200 2400
+Connection ~ 2200 2400
+Wire Wire Line
+	2200 2400 2150 2400
+Wire Wire Line
+	2200 1800 2200 1750
+Wire Wire Line
+	2200 1750 2050 1750
+Wire Wire Line
+	1750 1750 1550 1750
+Wire Wire Line
+	1550 1750 1550 1850
+NoConn ~ 900  3950
+NoConn ~ 1750 4900
+NoConn ~ 3150 5850
+NoConn ~ 2150 2600
+NoConn ~ 2150 2700
+NoConn ~ 2150 2800
+NoConn ~ 2650 3750
+NoConn ~ 3050 3750
 $EndSCHEMATC

Commit message: All parts except KC2016Z are associated with footprints now
Parts:
- C1, C2, C3, C4, C5, C6, C7, C8: footprint (none) -> Capacitor_SMD:C_0805_2012Metric
- D1: footprint (none) -> LED_SMD:LED_0805_2012Metric
- J1: footprint (none) -> Connector_USB:USB_Micro-B_Molex_47346-0001
- J2, J3: footprint (none) -> Connector_PinSocket_2.54mm:PinSocket_1x10_P2.54mm_Vertical
- J4: footprint (none) -> Connector_PinSocket_2.54mm:PinSocket_1x03_P2.54mm_Vertical
- JP1, JP2: footprint (none) -> Connector_PinSocket_2.54mm:PinSocket_1x02_P2.54mm_Vertical
- R1: footprint (none) -> Resistor_SMD:R_0805_2012Metric
- Y1: footprint (none) -> Custom:XTAL_ABS25-32.768KHZ-6-1-T
Changed lines of the file:
@@
 F 0 "C5" H 5028 1996 50  0000 L CNN
 F 1 "100nF" H 5028 1905 50  0000 L CNN
-F 2 "" H 4850 1950 50  0001 C CNN
+F 2 "Capacitor_SMD:C_0805_2012Metric" H 4850 1950 50  0001 C CNN
 F 3 "~" H 4850 1950 50  0001 C CNN
 	1    4850 1950
@@
 F 0 "C7" H 6178 1996 50  0000 L CNN
 F 1 "100nF" H 6178 1905 50  0000 L CNN
-F 2 "" H 6000 1950 50  0001 C CNN
+F 2 "Capacitor_SMD:C_0805_2012Metric" H 6000 1950 50  0001 C CNN
 F 3 "~" H 6000 1950 50  0001 C CNN
 	1    6000 1950
@@
 F 0 "C8" H 6678 1996 50  0000 L CNN
 F 1 "1uF" H 6678 1905 50  0000 L CNN
-F 2 "" H 6500 1950 50  0001 C CNN
+F 2 "Capacitor_SMD:C_0805_2012Metric" H 6500 1950 50  0001 C CNN
 F 3 "~" H 6500 1950 50  0001 C CNN
 	1    6500 1950
@@
 F 0 "C6" H 5478 1996 50  0000 L CNN
 F 1 "10uF" H 5478 1905 50  0000 L CNN
-F 2 "" H 5300 1950 50  0001 C CNN
+F 2 "Capacitor_SMD:C_0805_2012Metric" H 5300 1950 50  0001 C CNN
 F 3 "~" H 5300 1950 50  0001 C CNN
 	1    5300 1950
@@
 F 0 "J1" H 1907 3067 50  0000 C CNN
 F 1 "USB_B_Micro" H 1907 2976 50  0000 C CNN
-F 2 "" H 2000 2550 50  0001 C CNN
+F 2 "Connector_USB:USB_Micro-B_Molex_47346-0001" H 2000 2550 50  0001 C CNN
 F 3 "~" H 2000 2550 50  0001 C CNN
 	1    1850 2600
@@
 F 0 "J4" H 7958 3081 50  0000 C CNN
 F 1 "Conn_01x03_Male" H 7958 2990 50  0000 C CNN
-F 2 "" H 7850 2800 50  0001 C CNN
+F 2 "Connector_PinSocket_2.54mm:PinSocket_1x03_P2.54mm_Vertical" H 7850 2800 50  0001 C CNN
 F 3 "~" H 7850 2800 50  0001 C CNN
 	1    7850 2800
@@
 F 0 "Y1" V 2804 3994 50  0000 L CNN
 F 1 "ABS25-32.768KHZ-6-T" V 2895 3994 50  0000 L CNN
-F 2 "" H 2850 3750 50  0001 C CNN
+F 2 "Custom:XTAL_ABS25-32.768KHZ-6-1-T" H 2850 3750 50  0001 C CNN
 F 3 "~" H 2850 3750 50  0001 C CNN
 	1    2850 3750
@@
 F 0 "C1" V 1985 3450 50  0000 C CNN
 F 1 "4.3pF" V 2076 3450 50  0000 C CNN
-F 2 "" H 2300 3450 50  0001 C CNN
+F 2 "Capacitor_SMD:C_0805_2012Metric" H 2300 3450 50  0001 C CNN
 F 3 "~" H 2300 3450 50  0001 C CNN
 	1    2300 3450
@@
 F 0 "C2" V 1985 4150 50  0000 C CNN
 F 1 "4.3pF" V 2076 4150 50  0000 C CNN
-F 2 "" H 2300 4150 50  0001 C CNN
+F 2 "Capacitor_SMD:C_0805_2012Metric" H 2300 4150 50  0001 C CNN
 F 3 "~" H 2300 4150 50  0001 C CNN
 	1    2300 4150
@@
 F 0 "J3" H 6308 5981 50  0000 C CNN
 F 1 "Conn_01x10_Male" H 6308 5890 50  0000 C CNN
-F 2 "" H 6200 5400 50  0001 C CNN
+F 2 "Connector_PinSocket_2.54mm:PinSocket_1x10_P2.54mm_Vertical" H 6200 5400 50  0001 C CNN
 F 3 "~" H 6200 5400 50  0001 C CNN
 	1    6200 5400
@@
 F 0 "J2" H 3058 6031 50  0000 C CNN
 F 1 "Conn_01x10_Male" H 3058 5940 50  0000 C CNN
-F 2 "" H 2950 5450 50  0001 C CNN
+F 2 "Connector_PinSocket_2.54mm:PinSocket_1x10_P2.54mm_Vertical" H 2950 5450 50  0001 C CNN
 F 3 "~" H 2950 5450 50  0001 C CNN
 	1    2950 5450
@@
 F 0 "JP2" H 3500 4414 50  0000 C CNN
 F 1 "Jumper" H 3500 4323 50  0000 C CNN
-F 2 "" H 3500 4150 50  0001 C CNN
+F 2 "Connector_PinSocket_2.54mm:PinSocket_1x02_P2.54mm_Vertical" H 3500 4150 50  0001 C CNN
 F 3 "~" H 3500 4150 50  0001 C CNN
 	1    3500 4150
@@
 F 0 "JP1" H 3500 3714 50  0000 C CNN
 F 1 "Jumper" H 3500 3623 50  0000 C CNN
-F 2 "" H 3500 3450 50  0001 C CNN
+F 2 "Connector_PinSocket_2.54mm:PinSocket_1x02_P2.54mm_Vertical" H 3500 3450 50  0001 C CNN
 F 3 "~" H 3500 3450 50  0001 C CNN
 	1    3500 3450
@@
 F 0 "C3" H 2678 1946 50  0000 L CNN
 F 1 "4.7u" H 2678 1855 50  0000 L CNN
-F 2 "" H 2500 1900 50  0001 C CNN
+F 2 "Capacitor_SMD:C_0805_2012Metric" H 2500 1900 50  0001 C CNN
 F 3 "~" H 2500 1900 50  0001 C CNN
 	1    2500 1900
@@
 F 0 "C4" H 3628 1946 50  0000 L CNN
 F 1 "4.7u" H 3628 1855 50  0000 L CNN
-F 2 "" H 3450 1900 50  0001 C CNN
+F 2 "Capacitor_SMD:C_0805_2012Metric" H 3450 1900 50  0001 C CNN
 F 3 "~" H 3450 1900 50  0001 C CNN
 	1    3450 1900
@@
 F 0 "R1" H 2268 1996 50  0000 L CNN
 F 1 "200" H 2268 1905 50  0000 L CNN
-F 2 "" V 2240 1940 50  0001 C CNN
+F 2 "Resistor_SMD:R_0805_2012Metric" V 2240 1940 50  0001 C CNN
 F 3 "~" H 2200 1950 50  0001 C CNN
 	1    2200 1950
@@
 F 0 "D1" H 1893 1967 50  0000 C CNN
 F 1 "LED" H 1893 1876 50  0000 C CNN
-F 2 "" H 1900 1750 50  0001 C CNN
+F 2 "LED_SMD:LED_0805_2012Metric" H 1900 1750 50  0001 C CNN
 F 3 "~" H 1900 1750 50  0001 C CNN
 	1    1900 1750
