File: hw/designs/stm32_breakout/stm32_breakout.sch (KiCad schematic (older format))
At the start: 16 parts, among them J1 USB_B_Micro, J2 Conn_01x10_Male, J3 Conn_01x10_Male, U1 AP7361C-33E, U2 STM32L031F6Px, U3 KC2016Z

Commit message: Attempt to switch the pinout of the regulator part. Made a new project specific library called Adek lib
Parts:
- U1: value AP7361C-33E -> AP7361C-33ER; symbol Regulator_Linear:AP7361C-33E -> AdekLib:AP7361C-33ER
Connections:
- net +3V3: now also U1.2 (VO); no longer U1.3 (VO)
- net GND: now also U1.1 (GND); no longer U1.2 (GND)
- net at C1.2, J1.1 (VBUS), R1.2: now also U1.3 (VI); no longer U1.1 (VI)
Changed lines of the file:
@@
-	1    0    0    -1
-$EndComp
-$Comp
-L Regulator_Linear:AP7361C-33E U1
-U 1 1 608118E6
-P 3000 2400
-F 0 "U1" H 3000 2642 50  0000 C CNN
-F 1 "AP7361C-33E" H 3000 2551 50  0000 C CNN
-F 2 "Package_TO_SOT_SMD:SOT-223-3_TabPin2" H 3000 2625 50  0001 C CIN
-F 3 "https://www.diodes.com/assets/Datasheets/AP7361C.pdf" H 3000 2350 50  0001 C CNN
-	1    3000 2400
 	1    0    0    -1
 $EndComp
@@
 	1850 3100 1800 3100
 Connection ~ 1800 3100
-Wire Wire Line
-	2700 2400 2500 2400
 Wire Wire Line
 	7150 3600 7150 2750
@@
 Connection ~ 5300 2400
 Wire Wire Line
-	3300 2400 3450 2400
-Wire Wire Line
 	3450 2400 3450 2150
 Wire Wire Line
 	3450 2400 4000 2400
-Connection ~ 3450 2400
 Wire Wire Line
 	2500 2150 2500 2400
@@
 Text Notes 8200 2200 0    50   ~ 0
 Use KC2016Z: R2 = 0, R3 = UNPOP\nUse Internal Clock: R2 = UNPOP, R3 = 0
+Connection ~ 3450 2400
+Wire Wire Line
+	3300 2400 3450 2400
+Wire Wire Line
+	2700 2400 2500 2400
+$Comp
+L AdekLib:AP7361C-33ER U1
+U 1 1 608118E6
+P 3000 2250
+F 0 "U1" H 3000 2492 50  0000 C CNN
+F 1 "AP7361C-33ER" H 3000 2401 50  0000 C CNN
+F 2 "Package_TO_SOT_SMD:SOT-223-3_TabPin2" H 3000 2475 50  0001 C CIN
+F 3 "https://www.diodes.com/assets/Datasheets/AP7361C.pdf" H 3000 2200 50  0001 C CNN
+	1    3000 2250
+	1    0    0    -1
+$EndComp
 $EndSCHEMATC
