File: hw/designs/stm32_breakout/rev1/stm32_breakout.sch (KiCad schematic (older format))
At the start: 17 parts, among them J1 USB_B_Micro, J2 Conn_01x10_Male, J3 Conn_01x10_Male, U1 LM3670MF, U2 STM32L031F6Px, U3 KC2016Z

Commit message: tried to add part links and data sheets but my gitignore doesn't seem to be working
Parts:
- D1: PartLink (none) -> https://www.digikey.comproducts/detail/american-opto-plus-l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
Changed lines of the file:
@@
 F 1 "LED" H 1343 1876 50  0000 C CNN
 F 2 "LED_SMD:LED_0805_2012Metric" H 1350 1750 50  0001 C CNN
-F 3 "~" H 1350 1750 50  0001 C CNN
+F 3 "https://www.aopled.com/AOP_PDFs/L171L-LPGC.pdf" H 1350 1750 50  0001 C CNN
+F 4 "https://www.digikey.comproducts/detail/american-opto-plus-led/L171L-LPGC/12325399" H 1350 1750 50  0001 C CNN "PartLink"
 	1    1350 1750
 	1    0    0    -1
