File: hw/designs/stm32_breakout/rev1/stm32_breakout.sch (KiCad schematic (older format))
At the start: 17 parts, among them J1 USB_B_Micro, J2 Conn_01x10_Male, J3 Conn_01x10_Male, U1 LM3670MF, U2 STM32L031F6Px, U3 KC2016Z

Commit message: Updated with SWD pins
Connections:
- net PA13 renamed PA13-SWDIO
- net PA14 renamed PA14-SWCLK
Changed lines of the file:
@@
 PA10
 Text Label 6700 3750 0    50   ~ 0
-PA13
+PA13-SWDIO
 Text Label 6700 3850 0    50   ~ 0
-PA14
+PA14-SWCLK
 $Comp
 L power:GND #PWR08
@@
 PA9
 Text Label 3650 5550 0    50   ~ 0
-PA13
+PA13-SWDIO
 Text Label 3650 5650 0    50   ~ 0
-PA14
+PA14-SWCLK
 Wire Wire Line
 	6400 5100 6950 5100
