File: hw/designs/keyboard/keyboard/keyboard.kicad_pcb (KiCad board)
At the start: 2 copper layers, 25 parts, among them J1 Conn_01x08_Female, Q1 2N2222A, Q2 2N2222A, Q3 2N2222A, Q4 2N2222A, Q5 2N2222A, Q6 2N2222A, Q7 2N2222A, Q8 2N2222A

Commit message: Adding sheets
Parts:
- added D10: 1N4007, Diode_THT:D_DO-41_SOD81_P10.16mm_Horizontal, F.Cu at (20.8, 62.2)
- added D11: 1N4007, Diode_THT:D_DO-41_SOD81_P10.16mm_Horizontal, F.Cu at (20.8, 58.0)
- added D12: 1N4007, Diode_THT:D_DO-41_SOD81_P10.16mm_Horizontal, F.Cu at (34.7, 53.7)
- added D13: 1N4007, Diode_THT:D_DO-41_SOD81_P10.16mm_Horizontal, F.Cu at (20.8, 53.7)
- added D14: 1N4007, Diode_THT:D_DO-41_SOD81_P10.16mm_Horizontal, F.Cu at (34.7, 49.5)
- added D15: 1N4007, Diode_THT:D_DO-41_SOD81_P10.16mm_Horizontal, F.Cu at (20.8, 49.5)
- added D16: 1N4007, Diode_THT:D_DO-41_SOD81_P10.16mm_Horizontal, F.Cu at (16.2, 71.9)
- added D9: 1N4007, Diode_THT:D_DO-41_SOD81_P10.16mm_Horizontal, F.Cu at (20.8, 66.5)
- added J2: Conn_01x08_Female, Connector_PinSocket_2.54mm:PinSocket_1x08_P2.54mm_Vertical, F.Cu at (16.7, 49.7)
- added Q10: 2N2222A, Package_TO_SOT_THT:TO-92_Inline, F.Cu at (56.8, 70.3)
- added Q11: 2N2222A, Package_TO_SOT_THT:TO-92_Inline, F.Cu at (54.6, 64.5)
- added Q12: 2N2222A, Package_TO_SOT_THT:TO-92_Inline, F.Cu at (62.0, 56.4)
- added Q13: 2N2222A, Package_TO_SOT_THT:TO-92_Inline, F.Cu at (62.0, 50.6)
- added Q14: 2N2222A, Package_TO_SOT_THT:TO-92_Inline, F.Cu at (48.1, 64.5)
- added Q15: 2N2222A, Package_TO_SOT_THT:TO-92_Inline, F.Cu at (55.2, 58.7)
- added Q16: 2N2222A, Package_TO_SOT_THT:TO-92_Inline, F.Cu at (48.7, 58.7)
- added Q9: 2N2222A, Package_TO_SOT_THT:TO-92_Inline, F.Cu at (61.2, 64.5)
- added R10: 1k, Resistor_THT:R_Axial_DIN0207_L6.3mm_D2.5mm_P10.16mm_Horizontal, F.Cu at (43.1, 70.0)
- added R11: 1k, Resistor_THT:R_Axial_DIN0207_L6.3mm_D2.5mm_P10.16mm_Horizontal, F.Cu at (29.8, 74.7)
- added R12: 1k, Resistor_THT:R_Axial_DIN0207_L6.3mm_D2.5mm_P10.16mm_Horizontal, F.Cu at (34.4, 66.0)
- added R13: 1k, Resistor_THT:R_Axial_DIN0207_L6.3mm_D2.5mm_P10.16mm_Horizontal, F.Cu at (48.3, 53.4)
- added R14: 1k, Resistor_THT:R_Axial_DIN0207_L6.3mm_D2.5mm_P10.16mm_Horizontal, F.Cu at (48.3, 49.4)
- added R15: 1k, Resistor_THT:R_Axial_DIN0207_L6.3mm_D2.5mm_P10.16mm_Horizontal, F.Cu at (34.4, 61.9)
- added R16: 1k, Resistor_THT:R_Axial_DIN0207_L6.3mm_D2.5mm_P10.16mm_Horizontal, F.Cu at (34.4, 57.9)
- added R9: 1k, Resistor_THT:R_Axial_DIN0207_L6.3mm_D2.5mm_P10.16mm_Horizontal, F.Cu at (29.8, 70.6)
- R1, R2, R3, R4, R5, R6, R7, R8: value R -> 1k
- moved D2 136.9 mm to (20.8, 33.6), turned to 0 degrees
- moved D1 121.3 mm to (16.2, 39.0), turned to 0 degrees
- moved R2 114.7 mm to (43.1, 37.2), turned to 0 degrees
- moved R1 109.8 mm to (34.4, 33.1), turned to 0 degrees
- moved Q2 108.6 mm to (56.8, 37.4)
- moved Q1 98.4 mm to (61.2, 31.6)
- moved D3 97.1 mm to (20.8, 16.6)
- moved D5 96.0 mm to (20.8, 20.9)
- moved R3 92.5 mm to (29.8, 41.8)
- moved Q5 90.8 mm to (62.0, 17.7)
- moved R7 88.6 mm to (34.4, 29.1)
- moved Q8 87.0 mm to (48.7, 25.8)
- moved Q6 86.9 mm to (48.1, 31.6)
- moved D7 86.3 mm to (20.8, 25.1)
- moved D8 86.3 mm to (20.8, 29.4)
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Connections:
- net /BASE_ROW1_COL1 renamed /ROW1_COL[1-8]/BASE_ROW1_COL1
- net /BASE_ROW1_COL2 renamed /ROW1_COL[1-8]/BASE_ROW1_COL2
- net /BASE_ROW1_COL3 renamed /ROW1_COL[1-8]/BASE_ROW1_COL3
- net /BASE_ROW1_COL4 renamed /ROW1_COL[1-8]/BASE_ROW1_COL4
- net /BASE_ROW1_COL5 renamed /ROW1_COL[1-8]/BASE_ROW1_COL5
- net /BASE_ROW1_COL6 renamed /ROW1_COL[1-8]/BASE_ROW1_COL6
- net /BASE_ROW1_COL7 renamed /ROW1_COL[1-8]/BASE_ROW1_COL7
- net /BASE_ROW1_COL8 renamed /ROW1_COL[1-8]/BASE_ROW1_COL8
- net /COLLECTOR_ROW1_COL1 renamed /ROW1_COL[1-8]/COLLECTOR_ROW1_COL1
- net /COLLECTOR_ROW1_COL2 renamed /ROW1_COL[1-8]/COLLECTOR_ROW1_COL2
- net /COLLECTOR_ROW1_COL3 renamed /ROW1_COL[1-8]/COLLECTOR_ROW1_COL3
- net /COLLECTOR_ROW1_COL4 renamed /ROW1_COL[1-8]/COLLECTOR_ROW1_COL4
- net /COLLECTOR_ROW1_COL5 renamed /ROW1_COL[1-8]/COLLECTOR_ROW1_COL5
- net /COLLECTOR_ROW1_COL6 renamed /ROW1_COL[1-8]/COLLECTOR_ROW1_COL6
- net /COLLECTOR_ROW1_COL7 renamed /ROW1_COL[1-8]/COLLECTOR_ROW1_COL7
- net /COLLECTOR_ROW1_COL8 renamed /ROW1_COL[1-8]/COLLECTOR_ROW1_COL8
- net /ENABLE_ROW1_COL1 renamed /ROW1_COL[1-8]/ENABLE_ROW1_COL1
- net /ENABLE_ROW1_COL2 renamed /ROW1_COL[1-8]/ENABLE_ROW1_COL2
- net /ENABLE_ROW1_COL3 renamed /ROW1_COL[1-8]/ENABLE_ROW1_COL3
- net /ENABLE_ROW1_COL4 renamed /ROW1_COL[1-8]/ENABLE_ROW1_COL4
- net /ENABLE_ROW1_COL5 renamed /ROW1_COL[1-8]/ENABLE_ROW1_COL5
- net /ENABLE_ROW1_COL6 renamed /ROW1_COL[1-8]/ENABLE_ROW1_COL6
- net /ENABLE_ROW1_COL7 renamed /ROW1_COL[1-8]/ENABLE_ROW1_COL7
- net /ENABLE_ROW1_COL8 renamed /ROW1_COL[1-8]/ENABLE_ROW1_COL8
- net /ROW1 renamed ROW1
Routing:
- net /ROW1_COL1_EN: track 35.2 -> 0.00 mm
